Commit message: Front and Back gpu_lidar added

File: antobot_sim_description/urdf/c16.urdf.xacro (robot description, xacro)
@@ -11,5 +11,5 @@
         <parent link="laser_link_${position}_static"/>
         <child link="laser_link_${position}_frame"/>
-        <origin xyz="0 0 -0.046093" rpy="0 0 0"/>
+        <origin xyz="0 0 -0.046093" rpy="0 0 3.14"/>  <!-- The gpu_lidar sensor's lidar frame has to be 180 deg rotated  -->
     </joint>
     <!-- The lidar frame position - for visualisation -->
@@ -43,41 +43,43 @@
     </xacro:if>
     <gazebo reference="laser_link_${position}_static">
-      <sensor type="ray" name="lidar_${position}">
-        <always_on>true</always_on>
-        <pose>0 0 0 0 0 0</pose>
-        <visualize>false</visualize>
-        <update_rate>5</update_rate>
-        <ray>
-          <scan>
-            <horizontal>
-              <samples>1000</samples>
-              <resolution>1</resolution>
-              <min_angle>0</min_angle>
-              <max_angle>6.28318</max_angle>
-            </horizontal>
-            <vertical>
-              <samples>16</samples>
-              <resolution>1</resolution>
-              <min_angle>-0.2618</min_angle>
-              <max_angle>0.2618</max_angle>
-            </vertical>
-          </scan>
-            <range>
-            <min>0.4</min>
-            <max>20</max>
-            <resolution>0.01</resolution>
-          </range>
-        </ray>
-        <!--
-        <plugin name="plugin_1" filename="libgazebo_ros_velodyne_laser.so">
-            <gaussianNoise>0.00</gaussianNoise>
-            <alwaysOn>true</alwaysOn>
-            <updateRate>5</updateRate>
-            <topicName>/lidar_${position}/lslidar_point_cloud</topicName>
-            <frameName>laser_link_${position}</frameName>
-        </plugin>
-        -->
+      <sensor name='lidar_${position}' type='gpu_lidar'>"
+          <pose relative_to='laser_link_${position}_frame'>0 0 0 0 0 0</pose>
+          <ignition_frame_id>laser_link_${position}_frame</ignition_frame_id>
+          <topic>/antobot_ant/scan/${position}</topic>
+          <update_rate>10</update_rate>
+          <ray>
+              <scan>
+                  <horizontal>
+                      <samples>640</samples>
+                      <resolution>1</resolution>
+                      <min_angle>-1.396263</min_angle>
+                      <max_angle>1.396263</max_angle>
+                  </horizontal>
+                  <vertical>
+                      <samples>1</samples>
+                      <resolution>0.01</resolution>
+                      <min_angle>0</min_angle>
+                      <max_angle>0</max_angle>
+                  </vertical>
+              </scan>
+              <range>
+                  <min>0.5</min>
+                  <max>10.0</max>
+                  <resolution>0.01</resolution>
+              </range>
+          </ray>
+          <always_on>1</always_on>
+          <visualize>true</visualize>
       </sensor>
     </gazebo>
   </xacro:macro>
 </robot>
+<!--
+<plugin name="plugin_1" filename="libgazebo_ros_velodyne_laser.so">
+    <gaussianNoise>0.00</gaussianNoise>
+    <alwaysOn>true</alwaysOn>
+    <updateRate>5</updateRate>
+    <topicName>/lidar_${position}/lslidar_point_cloud</topicName>
+    <frameName>laser_link_${position}</frameName>
+</plugin>
+-->
