Commit message: Fix joint state, TF error. Add IMU plugin

File: antobot_sim_description/urdf/ant_v4.urdf.xacro (robot description, xacro)
@@ -63,10 +63,14 @@
         <wheel_radius>0.3</wheel_radius>
         <odom_publish_frequency>1</odom_publish_frequency>
+        <publish_odom>true</publish_odom>
+        <odom_topic>/odom</odom_topic>
+        <odom_frame>odom</odom_frame>
+        <robot_base_frame>base_link</robot_base_frame>
         <max_linear_acceleration>1</max_linear_acceleration>
         <min_linear_acceleration>-1</min_linear_acceleration>
         <max_angular_acceleration>2</max_angular_acceleration>
         <min_angular_acceleration>-2</min_angular_acceleration>
-        <max_linear_velocity>0.5</max_linear_velocity>
-        <min_linear_velocity>-0.5</min_linear_velocity>
+        <max_linear_velocity>2.0</max_linear_velocity>
+        <min_linear_velocity>-2.0</min_linear_velocity>
         <max_angular_velocity>1</max_angular_velocity>
         <min_angular_velocity>-1</min_angular_velocity>
@@ -75,18 +79,4 @@
         filename="ignition-gazebo-joint-state-publisher-system"
         name="ignition::gazebo::systems::JointStatePublisher">
-      </plugin>
-      <plugin
-        filename="ignition-gazebo-pose-publisher-system"
-        name="ignition::gazebo::systems::PosePublisher">
-        <publish_link_pose>true</publish_link_pose>
-        <use_pose_vector_msg>true</use_pose_vector_msg>
-        <static_publisher>true</static_publisher>
-        <static_update_frequency>1</static_update_frequency>
-      </plugin>
-      <plugin
-        filename="ignition-gazebo-odometry-publisher-system"
-        name="ignition::gazebo::systems::OdometryPublisher">
-        <odom_frame>antobot_ant/odom</odom_frame>
-        <robot_base_frame>antobot_ant</robot_base_frame>
       </plugin>
     </gazebo>
@@ -200,21 +190,25 @@
     <link name="imu_frame">
       <inertial>
+        <origin xyz="0 0 0" rpy="0 0 0" />
         <mass value="0.270" />
-        <origin xyz="0 0 0" rpy="0 0 0" />
-        <inertia ixx="2.632e-4" ixy="0" ixz="0" iyy="2.632e-4" iyz="0" izz="1.62e-4" />
+        <inertia ixx="0.0002632" ixy="0.0" ixz="0.0" iyy="0.0002632" iyz="0.0" izz="0.000162" />
       </inertial>
     </link>
-    <!--
-    <gazebo>
-      <plugin name="imu_plugin" filename="libgazebo_ros_imu.so">
-        <alwaysOn>true</alwaysOn>
-        <bodyName>imu_frame</bodyName>
-        <topicName>/imu/data</topicName>
-        <serviceName>imu_service</serviceName>
-        <gaussianNoise>0.0</gaussianNoise>
-        <updateRate>20.0</updateRate>
-      </plugin>
-    </gazebo>
-    -->
+    <gazebo reference="imu_frame">
+      <sensor type="imu" name="imu_sensor">
+        <always_on>true</always_on>
+        <update_rate>100.0</update_rate>
+        <visualize>true</visualize>
+        <imu>
+          <topic>/imu/data</topic>
+          <orientation_reference_frame>ENU</orientation_reference_frame>
+        </imu>
+        <plugin name="ignition::gazebo::systems::Imu"
+                filename="ignition-gazebo-imu-system">
+          <topic>/imu/data</topic>
+          <frame_id>imu_frame</frame_id>
+        </plugin>
+      </sensor>
+    </gazebo>
     <!-- Ultrasonics-->
     <!-- Actual sensors output on combined topic /antobridge/uss_dist -->
